File: MicroMod_STM32.kicad_pcb (KiCad board)
At the start: 2 copper layers, 21.2 x 0.6 mm, 21 parts, among them J1 M.2, U1 STM32F405RGTx, Y1 CSTNE8M00GH5L000R0

Commit message: update
Parts:
- removed C3: 4.7u, MicroMod_STM32:0402-TIGHT
- removed R1: 10k, MicroMod_STM32:0402-TIGHT
- C1, C5, C9: moved to B.Cu
- U1: footprint Package_QFP:LQFP-64_10x10mm_P0.5mm -> MicroMod_STM32:TQFP64
- moved C4 61.6 mm to (48.2, 72.0)
- moved R7 56.9 mm to (53.5, 62.2), turned to 270 degrees
- moved C10 47.7 mm to (48.2, 74.5), turned to 180 degrees
- moved R3 46.0 mm to (54.8, 62.2), turned to 270 degrees
- moved R4 45.9 mm to (64.2, 62.8), turned to 180 degrees
- moved C7 45.5 mm to (64.2, 64.0), turned to 180 degrees
- moved R2 42.2 mm to (56.0, 62.2), turned to 270 degrees
- moved C8 41.1 mm to (48.2, 73.2), turned to 180 degrees
- moved Y1 39.7 mm to (48.0, 69.2), turned to 270 degrees
- moved C6 37.8 mm to (52.2, 62.2), turned to 90 degrees
- moved R6 36.7 mm to (65.5, 70.8), turned to 180 degrees
- moved C5 36.0 mm to (54.2, 73.4), turned to 90 degrees
- moved R5 35.7 mm to (65.5, 72.0), turned to 180 degrees
- moved C9 33.7 mm to (59.5, 73.5), turned to 90 degrees
- moved C1 29.0 mm to (58.2, 73.5), turned to 90 degrees
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Connections:
- J1 pad 1: Net-(J1-Pad1) -> /VCC
- J1 pad 10: Net-(J1-Pad10) -> /C8
- J1 pad 11: Net-(J1-Pad11) -> /IMU_SDA
- J1 pad 12: Net-(J1-Pad12) -> /B12
- J1 pad 13: Net-(J1-Pad13) -> /IMU_SCL
- J1 pad 15: Net-(J1-Pad15) -> /SPI2_CLK
- J1 pad 17: Net-(J1-Pad17) -> /SPI2_MISO
- J1 pad 19: Net-(J1-Pad19) -> /SPI2_MOSI
- J1 pad 2: Net-(J1-Pad2) -> /VCC
- J1 pad 21: Net-(J1-Pad21) -> /MOTOR2
- J1 pad 3: Net-(J1-Pad3) -> /OTG_FS_D+
- J1 pad 33: Net-(J1-Pad33) -> GND
- J1 pad 35: Net-(J1-Pad35) -> /INT_GYR
- J1 pad 4: Net-(J1-Pad4) -> GND
- J1 pad 5: Net-(J1-Pad5) -> /OTG_FS_D-
- J1 pad 6: Net-(J1-Pad6) -> /NRF_TX
- J1 pad 68: Net-(J1-Pad68) -> /BOOT0
- J1 pad 7: Net-(J1-Pad7) -> /OTG_FS_ID
- J1 pad 70: Net-(J1-Pad70) -> /NRST
- J1 pad 72: Net-(J1-Pad72) -> /MOTOR4
- J1 pad 73: Net-(J1-Pad73) -> /VBAT
- J1 pad 74: Net-(J1-Pad74) -> GND
- J1 pad 75: Net-(J1-Pad75) -> /VCC
- J1 pad 8: Net-(J1-Pad8) -> /NRF_RX
- J1 pad 9: Net-(J1-Pad9) -> /OTG_FS_VBUS
Routing:
- net /VCC: track 0.00 -> 29.6 mm, vias 0 -> 1
- net /BOOT0: track 0.00 -> 21.9 mm, vias 0 -> 2
- net /INT_GYR: track 0.00 -> 19.5 mm, vias 0 -> 2
- net /MOTOR4: track 0.00 -> 18.8 mm, vias 0 -> 2
- net /VBAT: track 0.00 -> 18.0 mm, vias 0 -> 2
- net /OTG_FS_D+: track 0.00 -> 15.9 mm, vias 0 -> 2
- net /MOTOR3: track 0.00 -> 15.1 mm, vias 0 -> 1
- net /OTG_FS_D-: track 0.00 -> 14.9 mm, vias 0 -> 2
- net /OTG_FS_ID: track 0.00 -> 14.3 mm, vias 0 -> 2
- net /NRST: track 0.00 -> 13.8 mm, vias 0 -> 1
- net /IMU_SCL: track 0.00 -> 13.5 mm, vias 0 -> 2
- net /OTG_FS_VBUS: track 0.00 -> 12.9 mm, vias 0 -> 2
- net /IMU_SDA: track 0.00 -> 12.9 mm
- net /C8: track 0.00 -> 11.3 mm, vias 0 -> 1
- net /NRF_TX: track 0.00 -> 10.3 mm, vias 0 -> 1
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Other:
- board size 21.2 x 0.6 mm -> 22 x 22 mm
- copper layers 2 -> 4
- net class Default: clearance 0.2 -> 0.12; trace_width 0.25 -> 0.2
- rule trace_clearance: 0.2 -> 0.12
- rule trace_min: 0.2 -> 0.15

Commit message: version 1
Parts:
- added CON1: SM06B-SRSS-TB, MicroMod_STM32:SM06B, B.Cu at (50.2, 63.0)
- moved D1 0.35 mm to (64.8, 61.6)
- moved C5 0.30 mm to (54.0, 73.4)
- moved C10 0.25 mm to (48.0, 74.5)
- moved C4 0.25 mm to (48.0, 72.0)
- moved C8 0.25 mm to (48.0, 73.2)
- moved R4 0.20 mm to (64.2, 63.0)
- moved C7 0.10 mm to (64.2, 64.1)
Connections:
- J1 pad 14: Net-(J1-Pad14) -> /MOTOR1
- J1 pad 16: Net-(J1-Pad16) -> /NRF_CTRL
- J1 pad 18: Net-(J1-Pad18) -> GND
- J1 pad 20: Net-(J1-Pad20) -> /GREEN_R
- J1 pad 22: Net-(J1-Pad22) -> /RED_R
- J1 pad 23: Net-(J1-Pad23) -> /B10
- J1 pad 32: Net-(J1-Pad32) -> /B4
- J1 pad 34: Net-(J1-Pad34) -> /E_SPI_MOSI
- J1 pad 36: Net-(J1-Pad36) -> /E_SPI_MISO
- J1 pad 37: Net-(J1-Pad37) -> /B1
- J1 pad 38: Net-(J1-Pad38) -> /E_SPI_CLK
- J1 pad 39: Net-(J1-Pad39) -> /B0
- J1 pad 40: Net-(J1-Pad40) -> /E_SCL
- J1 pad 41: Net-(J1-Pad41) -> /C5
- J1 pad 42: Net-(J1-Pad42) -> /E_SDA
- J1 pad 43: Net-(J1-Pad43) -> /C4
- J1 pad 44: Net-(J1-Pad44) -> /E_TX1
- J1 pad 45: Net-(J1-Pad45) -> /A0
- J1 pad 46: Net-(J1-Pad46) -> /E_RX1
- J1 pad 47: Net-(J1-Pad47) -> /C13
- J1 pad 48: Net-(J1-Pad48) -> /E_RX2
- J1 pad 49: Net-(J1-Pad49) -> /B5
- J1 pad 50: Net-(J1-Pad50) -> /E_TX2
- J1 pad 51: Net-(J1-Pad51) -> /B8
- J1 pad 52: Net-(J1-Pad52) -> /C12
- J1 pad 54: Net-(J1-Pad54) -> /C15
- J1 pad 59: Net-(J1-Pad59) -> /VCC
- J1 pad 61: Net-(J1-Pad61) -> /STM_SWCLK
- J1 pad 63: Net-(J1-Pad63) -> GND
- J1 pad 65: Net-(J1-Pad65) -> /STM_SWIO
- J1 pad 66: Net-(J1-Pad66) -> /GREEN_L
- J1 pad 67: Net-(J1-Pad67) -> /NRST
- J1 pad 68: /BOOT0 -> /RED_L
- J1 pad 69: Net-(J1-Pad69) -> /STM_SWO
- J1 pad 70: /NRST -> /BOOT0
- J1 pad 71: Net-(J1-Pad71) -> /MOTOR3
- U1 pad 52: /E_TX2 -> /E_RX1
Routing:
- net /VCC: track 29.6 -> 101.6 mm, vias 1 -> 9
- net /STM_SWCLK: track 0.00 -> 38.1 mm, vias 0 -> 4
- net GND: track 6.25 -> 44.1 mm, vias 0 -> 21
- net /STM_SWIO: track 0.00 -> 37.5 mm, vias 0 -> 4
- net /STM_SWO: track 0.00 -> 30.4 mm, vias 0 -> 3
- net /B5: track 0.00 -> 22.9 mm, vias 0 -> 2
- net /B8: track 0.00 -> 21.6 mm, vias 0 -> 2
- net /GREEN_R: track 0.00 -> 20.1 mm, vias 0 -> 1
- net /C12: track 0.00 -> 20.0 mm, vias 0 -> 1
- net /RED_R: track 0.00 -> 19.3 mm, vias 0 -> 1
- net /E_RX1: track 0.00 -> 19.1 mm, vias 0 -> 2
- net /E_TX1: track 0.00 -> 18.7 mm, vias 0 -> 2
- net /E_SDA: track 2.66 -> 19.7 mm, vias 0 -> 1
- net /E_SCL: track 2.35 -> 19.3 mm, vias 0 -> 1
- net /C13: track 0.00 -> 16.3 mm, vias 0 -> 2
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- added copper zone on B.Cu, net GND
- added copper zone on F.Cu, net GND
- added copper zone on In1.Cu, net GND
- added copper zone on In2.Cu, net GND
Other:
- net class Default: via_dia 0.8 -> 0.5; via_drill 0.4 -> 0.25
- rule via_min_drill: 0.3 -> 0.25
