File: MicroMod_STM32.kicad_pcb (KiCad board)
At the start: 4 copper layers, 22 x 22 mm, 20 parts, among them CON1 SM06B-SRSS-TB, J1 M.2, U1 STM32F405RGTx, Y1 CSTNE8M00GH5L000R0

Commit message: no track under oscillator
Routing:
- net /B8: track 21.6 -> 29.2 mm
- net /INT_GYR: track 23.3 -> 28.8 mm
- net /VBAT: track 17.9 -> 19.8 mm
- net GND: vias 21 -> 22

Commit message: update vbat line
Routing:
- net /VCC: track 101.6 -> 98.5 mm, vias 9 -> 10

Commit message: update vcc copper
Parts:
- moved C2 1.24 mm to (64.2, 64.0)
- moved C7 0.92 mm to (64.3, 65.0)
Connections:
- net /BOOT0 renamed /STM_BOOT0
- net /E_SPI_CLK renamed /E_SPI_SCK
- net /NRST renamed /STM_NRST
- net /SPI2_CLK renamed /SPI2_SCK
- net /VBAT renamed /VCC_NRF
Routing:
- net /VCC: track 98.5 -> 44.2 mm, vias 10 -> 11
- net Net-(C2-Pad1): track 4.01 -> 6.13 mm
- net /OTG_FS_D+: track 15.8 -> 16.4 mm
- net /OTG_FS_D-: track 14.9 -> 15.5 mm
- net GND: track 44.1 -> 43.7 mm, vias 22 -> 23
- added copper zone on In2.Cu, net /VCC
- removed copper zone on In2.Cu, net GND

Commit message: MOTOR4 -> PB10
Connections:
- J1 pad 23: /B10 -> /MOTOR4
- J1 pad 72: /MOTOR4 -> /B9
- U1 pad 29: /B10 -> /MOTOR4
- U1 pad 62: /MOTOR4 -> /B9
Routing:
- net /B9: track 0.00 -> 20.0 mm, vias 0 -> 2
- net /MOTOR4: track 20.0 -> 5.32 mm, vias 2 -> 0
- net /B10: track 5.32 -> 0.00 mm

Commit message: MOTOR2->PB10,MOTOR4->PB8
Connections:
- J1 pad 21: /MOTOR2 -> /B11
- J1 pad 23: /MOTOR4 -> /MOTOR2
- J1 pad 51: /B8 -> /MOTOR4
- U1 pad 29: /MOTOR4 -> /MOTOR2
- U1 pad 30: /MOTOR2 -> /B11
- U1 pad 61: /B8 -> /MOTOR4
Routing:
- net /B8: track 29.2 -> 0.00 mm, vias 2 -> 0
- net /MOTOR4: track 5.32 -> 29.2 mm, vias 0 -> 2
- net /B11: track 0.00 -> 4.79 mm
- net /MOTOR2: track 4.79 -> 5.32 mm
