File: MicroMod_STM32.sch (KiCad schematic (older format))
At the start: 21 parts, among them J1 M.2, U1 STM32F405RGTx, Y1 CSTNE8M00GH5L000R0

Commit message: update
Parts:
- removed C3: 4.7u, MicroMod_STM32:0402-TIGHT, symbol Device:C
- removed R1: 10k, MicroMod_STM32:0402-TIGHT, symbol Device:R
- U1: footprint Package_QFP:LQFP-64_10x10mm_P0.5mm -> MicroMod_STM32:TQFP64
Connections:
- net B12: now also J1.12
- net BOOT0: now also J1.68
- net C8: now also J1.10
- net GND: now also J1.33, J1.4, J1.74
- net IMU_SCL: now also J1.13
- net IMU_SDA: now also J1.11
- net INT_GYR: now also J1.35
- net MOTOR2: now also J1.21
- net MOTOR4: now also J1.72
- net NRF_RX: now also J1.8
- net NRF_TX: now also J1.6
- net NRST: now also J1.70
- net OTG_FS_D+: now also J1.3
- net OTG_FS_D-: now also J1.5
- net OTG_FS_ID: now also J1.7
- net OTG_FS_VBUS: now also J1.9
- net SPI2_CLK: now also J1.15
- net SPI2_MISO: now also J1.17
- net SPI2_MOSI: now also J1.19
- net VBAT: now also J1.73
- net VCC: now also J1.1, J1.2, J1.75
Changed lines of the file:
@@
 F 0 "U1" H 3475 1486 50  0000 C CNN
 F 1 "STM32F405RGTx" H 3475 1395 50  0000 C CNN
-F 2 "Package_QFP:LQFP-64_10x10mm_P0.5mm" H 2875 1675 50  0001 R CNN
+F 2 "MicroMod_STM32:TQFP64" H 2875 1675 50  0001 R CNN
 F 3 "http://www.st.com/st-web-ui/static/active/en/resource/technical/document/datasheet/DM00037051.pdf" H 3475 3375 50  0001 C CNN
 	1    3475 3375
@@
 	2650 1350 2650 1275
 Connection ~ 2650 1275
-$Comp
-L Device:R R1
-U 1 1 61742E4E
-P 675 750
-F 0 "R1" H 745 796 50  0000 L CNN
-F 1 "10k" H 745 705 50  0000 L CNN
-F 2 "MicroMod_STM32:0402-TIGHT" V 605 750 50  0001 C CNN
-F 3 "~" H 675 750 50  0001 C CNN
-	1    675  750
-	1    0    0    -1
-$EndComp
-$Comp
-L Device:C C3
-U 1 1 61743219
-P 1025 750
-F 0 "C3" H 1140 796 50  0000 L CNN
-F 1 "4.7u" H 1140 705 50  0000 L CNN
-F 2 "MicroMod_STM32:0402-TIGHT" H 1063 600 50  0001 C CNN
-F 3 "~" H 1025 750 50  0001 C CNN
-	1    1025 750
-	1    0    0    -1
-$EndComp
 Text Label 2325 1975 0    50   ~ 0
 BOOT0
@@
 Wire Wire Line
 	4150 6675 4150 6825
+Text Label 6475 1975 2    50   ~ 0
+OTG_FS_D-
+Text Label 6475 1875 2    50   ~ 0
+OTG_FS_D+
+Text Label 6475 1775 2    50   ~ 0
+VCC
+$Comp
+L power:GND #PWR0109
+U 1 1 617812B4
+P 7475 1875
+F 0 "#PWR0109" H 7475 1625 50  0001 C CNN
+F 1 "GND" H 7480 1702 50  0000 C CNN
+F 2 "" H 7475 1875 50  0001 C CNN
+F 3 "" H 7475 1875 50  0001 C CNN
+	1    7475 1875
+	0    -1   -1   0
+$EndComp
+Text Label 6475 2075 2    50   ~ 0
+OTG_FS_ID
+Text Label 6475 2175 2    50   ~ 0
+OTG_FS_VBUS
+Text Label 6475 2275 2    50   ~ 0
+IMU_SDA
+Text Label 6475 2375 2    50   ~ 0
+IMU_SCL
+$Comp
+L power:GND #PWR0110
+U 1 1 61799E07
+P 6475 3075
+F 0 "#PWR0110" H 6475 2825 50  0001 C CNN
+F 1 "GND" H 6480 2902 50  0000 C CNN
+F 2 "" H 6475 3075 50  0001 C CNN
+F 3 "" H 6475 3075 50  0001 C CNN
+	1    6475 3075
+	0    1    1    0
+$EndComp
+Text Label 6475 5175 2    50   ~ 0
+VCC
+Text Label 7475 1775 0    50   ~ 0
+VCC
 $Comp
 L MicroMod_STM32:M.2 J1
@@
 	1    0    0    -1
 $EndComp
+Text Label 7475 1975 0    50   ~ 0
+NRF_TX
+Text Label 7475 2075 0    50   ~ 0
+NRF_RX
+Text Label 6475 2475 2    50   ~ 0
+SPI2_CLK
+Text Label 6475 2575 2    50   ~ 0
+SPI2_MISO
+Text Label 6475 2675 2    50   ~ 0
+SPI2_MOSI
+Text Label 6475 2775 2    50   ~ 0
+MOTOR2
+Text Label 6475 3175 2    50   ~ 0
+INT_GYR
+Text Label 7475 2175 0    50   ~ 0
+C8
+Text Label 7475 2275 0    50   ~ 0
+B12
+Text Label 6475 5075 2    50   ~ 0
+VBAT
+$Comp
+L power:GND #PWR0111
+U 1 1 61777529
+P 7475 5075
+F 0 "#PWR0111" H 7475 4825 50  0001 C CNN
+F 1 "GND" H 7480 4902 50  0000 C CNN
+F 2 "" H 7475 5075 50  0001 C CNN
+F 3 "" H 7475 5075 50  0001 C CNN
+	1    7475 5075
+	0    -1   -1   0
+$EndComp
+Text Label 7475 4975 0    50   ~ 0
+MOTOR4
+Text Label 7475 4875 0    50   ~ 0
+NRST
+Text Label 7475 4775 0    50   ~ 0
+BOOT0
 $EndSCHEMATC

Commit message: version 1
Parts:
- added CON1: SM06B-SRSS-TB, SM06B, symbol MicroMod_STM32:SM06B-SRSS-TB
Connections:
- net A0: now also J1.45
- net B0: now also J1.39
- net B1: now also J1.37
- net B10: now also J1.23
- net B4: now also J1.32
- net B5: now also J1.49
- net B8: now also J1.51
- net BOOT0: now also J1.70; no longer J1.68
- net C12: now also J1.52
- net C13: now also J1.47
- net C15: now also J1.54
- net C4: now also J1.43
- net C5: now also J1.41
- net E_RX2: now also J1.48
- net E_SCL: now also J1.40
- net E_SDA: now also J1.42
- net E_SPI_CLK: now also J1.38
- net E_SPI_MISO: now also J1.36
- net E_SPI_MOSI: now also J1.34
- net E_TX1: now also J1.44
- net E_TX2: now also J1.50; no longer U1.52 (PC11)
- net GND: now also J1.18, J1.63, CON1.3, CON1.G1, CON1.G2
- net GREEN_L: now also J1.66
- net GREEN_R: now also J1.20
- net MOTOR1: now also J1.14
- net MOTOR3: now also J1.71
- net NRF_CTRL: now also J1.16
- net NRST: now also J1.67, CON1.5; no longer J1.70
- net RED_L: now also J1.68
- net RED_R: now also J1.22
- net STM_SWCLK: now also J1.61, CON1.2
- net STM_SWIO: now also J1.65, CON1.4
- net STM_SWO: now also J1.69, CON1.6
- net VCC: now also J1.59, CON1.1
- net E_RX1: now reaches J1.46
- net E_RX1: now also U1.52 (PC11)
Changed lines of the file:
@@
 E_TX1
 Text Label 2775 4575 2    50   ~ 0
-E_TX2
+E_RX1
 Text Label 2775 4675 2    50   ~ 0
 C12
@@
 Text Label 7475 4975 0    50   ~ 0
 MOTOR4
+Text Label 6475 4775 2    50   ~ 0
+NRST
 Text Label 7475 4875 0    50   ~ 0
+BOOT0
+Text Label 7475 2975 0    50   ~ 0
+B4
+Text Label 7475 3075 0    50   ~ 0
+E_SPI_MOSI
+Text Label 7475 3175 0    50   ~ 0
+E_SPI_MISO
+Text Label 7475 3275 0    50   ~ 0
+E_SPI_CLK
+Text Label 7475 3375 0    50   ~ 0
+E_SCL
+Text Label 7475 3475 0    50   ~ 0
+E_SDA
+Text Label 6475 4975 2    50   ~ 0
+MOTOR3
+Text Label 7475 2375 0    50   ~ 0
+MOTOR1
+Text Label 6475 2875 2    50   ~ 0
+B10
+Text Label 7475 3575 0    50   ~ 0
+E_TX1
+Text Label 7475 3675 0    50   ~ 0
+E_RX1
+Text Label 6475 3275 2    50   ~ 0
+B1
+Text Label 6475 3375 2    50   ~ 0
+B0
+Text Label 7475 3775 0    50   ~ 0
+E_RX2
+Text Label 7475 3875 0    50   ~ 0
+E_TX2
+Text Label 7475 2475 0    50   ~ 0
+NRF_CTRL
+Text Label 6475 4875 2    50   ~ 0
+STM_SWO
+Text Label 6475 4675 2    50   ~ 0
+STM_SWIO
+Text Label 6475 4475 2    50   ~ 0
+STM_SWCLK
+$Comp
+L power:GND #PWR0112
+U 1 1 61763998
+P 6475 4575
+F 0 "#PWR0112" H 6475 4325 50  0001 C CNN
+F 1 "GND" H 6480 4402 50  0000 C CNN
+F 2 "" H 6475 4575 50  0001 C CNN
+F 3 "" H 6475 4575 50  0001 C CNN
+	1    6475 4575
+	0    1    1    0
+$EndComp
+Text Label 6475 3575 2    50   ~ 0
+C4
+Text Label 6475 3475 2    50   ~ 0
+C5
+Text Label 7475 4775 0    50   ~ 0
+RED_L
+Text Label 7475 4675 0    50   ~ 0
+GREEN_L
+Text Label 7475 2775 0    50   ~ 0
+RED_R
+Text Label 7475 2675 0    50   ~ 0
+GREEN_R
+Text Label 6475 3675 2    50   ~ 0
+A0
+Text Label 7475 4075 0    50   ~ 0
+C15
+Text Label 6475 3775 2    50   ~ 0
+C13
+Text Label 7475 3975 0    50   ~ 0
+C12
+Text Label 6475 3875 2    50   ~ 0
+B5
+Text Label 6475 3975 2    50   ~ 0
+B8
+$Comp
+L power:GND #PWR0113
+U 1 1 61789A89
+P 7475 2575
+F 0 "#PWR0113" H 7475 2325 50  0001 C CNN
+F 1 "GND" H 7480 2402 50  0000 C CNN
+F 2 "" H 7475 2575 50  0001 C CNN
+F 3 "" H 7475 2575 50  0001 C CNN
+	1    7475 2575
+	0    -1   -1   0
+$EndComp
+Text Label 3075 9150 2    50   ~ 0
+B8
+Text Label 6475 4375 2    50   ~ 0
+VCC
+$Comp
+L MicroMod_STM32:SM06B-SRSS-TB CON1
+U 1 1 6184116E
+P 9075 4400
+F 0 "CON1" H 9405 4693 50  0000 L CNN
+F 1 "SM06B-SRSS-TB" H 9075 4400 50  0001 L BNN
+F 2 "SM06B" H 9075 4400 50  0001 L BNN
+F 3 "" H 9075 4400 50  0001 L BNN
+F 4 "455-1806-1-ND" H 9075 4400 50  0001 L BNN "DIGIKEY#"
+F 5 "SM06B-SRSS-TB(LF)(SN)" H 9075 4400 50  0001 L BNN "MANF#"
+F 6 "JST Sales America Inc" H 9075 4400 50  0001 L BNN "MANF"
+	1    9075 4400
+	1    0    0    -1
+$EndComp
+$Comp
+L power:GND #PWR?
+U 1 1 6184376D
+P 9175 4500
+F 0 "#PWR?" H 9175 4250 50  0001 C CNN
+F 1 "GND" H 9180 4327 50  0000 C CNN
+F 2 "" H 9175 4500 50  0001 C CNN
+F 3 "" H 9175 4500 50  0001 C CNN
+	1    9175 4500
+	1    0    0    -1
+$EndComp
+Wire Wire Line
+	9275 4500 9175 4500
+Connection ~ 9175 4500
+Text Label 8975 4100 2    50   ~ 0
+STM_SWIO
+$Comp
+L power:GND #PWR?
+U 1 1 618473D8
+P 8975 4000
+F 0 "#PWR?" H 8975 3750 50  0001 C CNN
+F 1 "GND" H 8980 3827 50  0000 C CNN
+F 2 "" H 8975 4000 50  0001 C CNN
+F 3 "" H 8975 4000 50  0001 C CNN
+	1    8975 4000
+	0    1    1    0
+$EndComp
+Text Label 8975 3900 2    50   ~ 0
+STM_SWCLK
+Text Label 8975 3800 2    50   ~ 0
+VCC
+Text Label 8975 4300 2    50   ~ 0
+STM_SWO
+Text Label 8975 4200 2    50   ~ 0
 NRST
-Text Label 7475 4775 0    50   ~ 0
-BOOT0
 $EndSCHEMATC

Commit message: update vcc copper
Connections:
- net BOOT0 renamed STM_BOOT0
- net E_SPI_CLK renamed E_SPI_SCK
- net NRST renamed STM_NRST
- net SPI2_CLK renamed SPI2_SCK
- net VBAT renamed VCC_NRF
Changed lines of the file:
@@
 	2650 1350 2650 1275
 Connection ~ 2650 1275
-Text Label 2325 1975 0    50   ~ 0
-BOOT0
+Text Label 2325 1975 2    50   ~ 0
+STM_BOOT0
 Text Label 2650 1775 2    50   ~ 0
-NRST
+STM_NRST
 Wire Wire Line
 	4175 3675 4500 3675
@@
 C15
 Text Label 4175 4775 0    50   ~ 0
-SPI2_CLK
+SPI2_SCK
 Text Label 4175 4875 0    50   ~ 0
 SPI2_MISO
@@
 SPI2_MOSI
 Text Label 4175 2275 0    50   ~ 0
-E_SPI_CLK
+E_SPI_SCK
 Text Label 4175 2375 0    50   ~ 0
 E_SPI_MISO
@@
 B12
 Text Label 3275 1575 1    50   ~ 0
-VBAT
+VCC_NRF
 Wire Wire Line
 	3375 1575 3475 1575
@@
 NRF_RX
 Text Label 6475 2475 2    50   ~ 0
-SPI2_CLK
+SPI2_SCK
 Text Label 6475 2575 2    50   ~ 0
 SPI2_MISO
@@
 B12
 Text Label 6475 5075 2    50   ~ 0
-VBAT
+VCC_NRF
 $Comp
 L power:GND #PWR0111
@@
 MOTOR4
 Text Label 6475 4775 2    50   ~ 0
-NRST
+STM_NRST
 Text Label 7475 4875 0    50   ~ 0
-BOOT0
+STM_BOOT0
 Text Label 7475 2975 0    50   ~ 0
 B4
@@
 E_SPI_MISO
 Text Label 7475 3275 0    50   ~ 0
-E_SPI_CLK
+E_SPI_SCK
 Text Label 7475 3375 0    50   ~ 0
 E_SCL
@@
 STM_SWO
 Text Label 8975 4200 2    50   ~ 0
-NRST
+STM_NRST
 $EndSCHEMATC

Commit message: MOTOR4 -> PB10
Connections:
- net B10 is gone; now on net MOTOR4: J1.23, U1.29 (PB10)
- net MOTOR4: no longer J1.72, U1.62 (PB9)
- new net B9: J1.72, U1.62 (PB9)
Changed lines of the file:
@@
 B8
 Text Label 4175 4375 0    50   ~ 0
+B9
+Text Label 4175 4475 0    50   ~ 0
 MOTOR4
-Text Label 4175 4475 0    50   ~ 0
-B10
 Text Label 4175 4575 0    50   ~ 0
 MOTOR2
@@
 $EndComp
 Text Label 7475 4975 0    50   ~ 0
-MOTOR4
+B9
 Text Label 6475 4775 2    50   ~ 0
 STM_NRST
@@
 MOTOR1
 Text Label 6475 2875 2    50   ~ 0
-B10
+MOTOR4
 Text Label 7475 3575 0    50   ~ 0
 E_TX1

Commit message: MOTOR2->PB10,MOTOR4->PB8
Connections:
- net B8: no longer J1.51, U1.61 (PB8)
- net MOTOR2: now also J1.23, U1.29 (PB10); no longer J1.21, U1.30 (PB11)
- net MOTOR4: now also J1.51, U1.61 (PB8); no longer J1.23, U1.29 (PB10)
- new net B11: J1.21, U1.30 (PB11)
Changed lines of the file:
@@
 Text Label 4175 4175 0    50   ~ 0
 E_SDA
-Text Label 4175 4275 0    50   ~ 0
-B8
+Text Label 4175 4575 0    50   ~ 0
+B11
 Text Label 4175 4375 0    50   ~ 0
 B9
+Text Label 4175 4275 0    50   ~ 0
+MOTOR4
 Text Label 4175 4475 0    50   ~ 0
-MOTOR4
-Text Label 4175 4575 0    50   ~ 0
 MOTOR2
 Text Label 4175 4675 0    50   ~ 0
@@
 SPI2_MOSI
 Text Label 6475 2775 2    50   ~ 0
-MOTOR2
+B11
 Text Label 6475 3175 2    50   ~ 0
 INT_GYR
@@
 MOTOR1
 Text Label 6475 2875 2    50   ~ 0
-MOTOR4
+MOTOR2
 Text Label 7475 3575 0    50   ~ 0
 E_TX1
@@
 B5
 Text Label 6475 3975 2    50   ~ 0
-B8
+MOTOR4
 $Comp
 L power:GND #PWR0113
